File: coilSafety/coilSafety.kicad_sch (KiCad schematic)
At the start: 22 parts, among them J1 PJ-037BH, J10 Conn_01x02_Pin, J11 Conn_01x02_Pin, J2 Screw_Terminal_01x08, J3 Screw_Terminal_01x02, J4 Screw_Terminal_01x02, J5 Screw_Terminal_01x06, J6 Screw_Terminal_01x02, J7 Conn_01x01_Pin, J8 Conn_01x08_Pin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

Commit message: v2 schematic complete
Parts:
- removed J7: Conn_01x01_Pin, Connector_Samtec_HPM_THT:Samtec_HPM-01-01-x-S_Straight_1x01_Pitch5.08mm, symbol Connector:Conn_01x01_Pin
- removed J8: Conn_01x08_Pin, Connector_PinHeader_2.54mm:PinHeader_1x08_P2.54mm_Vertical, symbol Connector:Conn_01x08_Pin
- K1: footprint Footprints:AZ943-1CH-12DE -> AZ943-1CH_AMZ
- M1: value ~ -> ESP32-C6-DevKitM-1
- U1, U2: value ~ -> AZDC007-1AE-12D
Connections:
- net +3.3V: no longer PS3.2 (+VIN)
- net +5V: no longer M1.14 (5v)
- net GND: now also M1.30 (GND), PS1.1 (-VIN), PS2.1 (-VIN)
- net at J1.1, J9.2 (Pin_2): now also J6.1 (Pin_1); no longer K1.1
- net at J1.2: now also J9.1 (Pin_1), K1.1, K1.4; no longer J6.2 (Pin_2)
- net at J2.8 (Pin_8), R1.1: now also M1.3 (GPIO_2); no longer M1.6 (GPIO_5)
- net at J2.2 (Pin_2), R4.1: now also M1.6 (GPIO_5); no longer M1.10 (GPIO_6)
- net at J2.4 (Pin_4), R3.1: now also M1.5 (GPIO_4); no longer M1.8 (GPIO_1)
- net at J2.6 (Pin_6), R2.1: now also M1.4 (GPIO_3); no longer M1.7 (GPIO_0)
- net at K1.3: now also J6.2 (Pin_2)
- new net: M1.10 (GPIO_6), PS3.2 (+VIN)
Other:
- note added: "2x Moisture Sensor Terminal"
- note added: "Boost Converter"
- note added: "Coil 1 Terminal"
- note added: "Coil 2 Terminal"
- note added: "Coil Power Switch"
- note added: "Coil Short Pin"
- note added: "Moisture Sensor Connection"
- note added: "Power Relay"
- note added: "Pump In"
- note added: "Pump Out"
- note added: "Pump Short Pin"
- note added: "Thermistor Connection"
- note added: "Water Pump Power Switch"
- company: (none) -> Biedermann Lab
- title: (none) -> Coil Safety Circuit
- moved on the sheet: J1, J10, J11, J2, J3, J4, J5, J6, J9, K1, M1, PS1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

Commit message: Working on PCB
Parts:
- J10, J11, J9: footprint Connector_PinHeader_2.54mm:PinHeader_1x02_P2.54mm_Vertical -> TerminalBlock:TerminalBlock_bornier-2_P5.08mm
- K1: footprint AZ943-1CH_AMZ -> Footprints:AZ943-1CH-12DE
Connections:
- net +5V: now also M1.14 (5v)
Changed lines of the file:
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@@
+	(wire
+		(pts
+			(xy 102.87 116.84) (xy 102.87 115.57)
+		)
+		(stroke
+			(width 0)
+			(type default)
+		)
+	)
 	(wire
 		(pts
@@
 		(pts
 			(xy 87.63 68.58) (xy 87.63 73.66)
+		)
+		(stroke
+			(width 0)
+			(type default)
+		)
+	)
+	(wire
+		(pts
+			(xy 109.22 116.84) (xy 102.87 116.84)
 		)
 		(stroke
@@
 			)
 		)
-		(property "Footprint" "Connector_PinHeader_2.54mm:PinHeader_1x02_P2.54mm_Vertical"
+		(property "Footprint" "TerminalBlock:TerminalBlock_bornier-2_P5.08mm"
 			(at 67.31 148.59 0)
 			(effects
@@
 			)
 		)
-		(property "Footprint" "Connector_PinHeader_2.54mm:PinHeader_1x02_P2.54mm_Vertical"
+		(property "Footprint" "TerminalBlock:TerminalBlock_bornier-2_P5.08mm"
 			(at 237.49 16.51 0)
 			(effects
@@
 			)
 		)
-		(property "Footprint" "Connector_PinHeader_2.54mm:PinHeader_1x02_P2.54mm_Vertical"
+		(property "Footprint" "TerminalBlock:TerminalBlock_bornier-2_P5.08mm"
 			(at 245.11 22.86 0)
 			(effects
@@
 	)
 	(symbol
+		(lib_id "power:+5V")
+		(at 102.87 115.57 0)
+		(unit 1)
+		(exclude_from_sim no)
+		(in_bom yes)
+		(on_board yes)
+		(dnp no)
+		(fields_autoplaced yes)
+		(property "Reference" "#PWR011"
+			(at 102.87 119.38 0)
+			(effects
+				(font
+					(size 1.27 1.27)
+				)
+				(hide yes)
+			)
+		)
+		(property "Value" "+5V"
+			(at 102.87 110.49 0)
+			(effects
+				(font
+					(size 1.27 1.27)
+				)
+			)
+		)
+		(property "Footprint" ""
+			(at 102.87 115.57 0)
+			(effects
+				(font
+					(size 1.27 1.27)
+				)
+				(hide yes)
+			)
+		)
+		(property "Datasheet" ""
+			(at 102.87 115.57 0)
+			(effects
+				(font
+					(size 1.27 1.27)
+				)
+				(hide yes)
+			)
+		)
+		(property "Description" "Power symbol creates a global label with name \"+5V\""
+			(at 102.87 115.57 0)
+			(effects
+				(font
+					(size 1.27 1.27)
+				)
+				(hide yes)
+			)
+		)
+		(pin "1"
+		)
+		(instances
+			(project ""
+				(path "/81435b52-0125-497d-af5b-c0831d6a55aa"
+					(reference "#PWR011")
+					(unit 1)
+				)
+			)
+		)
+	)
+	(symbol
 		(lib_id "sensors:AZ943-1CH-12DE")
 		(at 67.31 172.72 0)
@@
 			)
 		)
-		(property "Footprint" "AZ943-1CH_AMZ"
+		(property "Footprint" "Footprints:AZ943-1CH-12DE"
 			(at 67.31 172.72 0)
 			(effects
